File: rest/rest.kicad_pcb (KiCad board)
At the start: 2 copper layers, 143 x 99.2 mm, 17 parts, among them J1 MJ-4PP-9

Commit message: update readme.
Parts:
- removed D1, D10, D11, D12, D2, D3, D4, D5, D6, D7, D8, D9: WS2812B, LED_SMD:LED_WS2812B_PLCC4_5.0x5.0mm_P3.2mm
- removed REF** (x4): MountingHole_2.2mm_M2_Pad_Via, MountingHole:MountingHole_2.2mm_M2_Pad_Via
- added J2: Conn_01x01, MountingHole:MountingHole_2.2mm_M2_Pad_Via, F.Cu at (37.0, 123.0)
- added J3: Conn_01x01, MountingHole:MountingHole_2.2mm_M2_Pad_Via, F.Cu at (37.0, 38.8)
- added J4: Conn_01x01, MountingHole:MountingHole_2.2mm_M2_Pad_Via, F.Cu at (136.5, 123.0)
- added J5: Conn_01x01, MountingHole:MountingHole_2.2mm_M2_Pad_Via, F.Cu at (167.0, 50.0)
- added L1: YS-SK6812MINI, Keyboard:YS-SK6812MINI-E-reverse, F.Cu at (127.0, 107.5)
- added L2: YS-SK6812MINI, Keyboard:YS-SK6812MINI-E-reverse, F.Cu at (93.3, 107.5)
- added L3: YS-SK6812MINI, Keyboard:YS-SK6812MINI-E-reverse, F.Cu at (57.2, 107.5)
- added L4: YS-SK6812MINI, Keyboard:YS-SK6812MINI-E-reverse, F.Cu at (57.2, 46.8)
- added L5: YS-SK6812MINI, Keyboard:YS-SK6812MINI-E-reverse, F.Cu at (91.4, 46.8)
- added L6: YS-SK6812MINI, Keyboard:YS-SK6812MINI-E-reverse, F.Cu at (127.0, 46.8)
- moved J1 111.0 mm to (150.5, 109.0), turned to 245.1 degrees
Routing:
- net GND: track 420.9 -> 849.9 mm
- net Net-(L3-Pad2): track 0.00 -> 126.9 mm
- net VCC: track 437.9 -> 509.2 mm
- net Net-(L2-Pad2): track 0.00 -> 63.6 mm
- net Net-(L5-Pad2): track 0.00 -> 62.4 mm
- net Net-(L4-Pad2): track 0.00 -> 59.8 mm
- net Net-(L1-Pad2): track 0.00 -> 58.6 mm
- net Net-(D10-Pad4): track 49.7 -> 0.00 mm
- net Net-(D3-Pad2): track 48.5 -> 0.00 mm
- net Net-(D8-Pad2): track 33.1 -> 0.00 mm
- net Net-(D2-Pad2): track 33.1 -> 0.00 mm
- net Net-(D5-Pad2): track 32.4 -> 0.00 mm
- net Net-(D11-Pad2): track 32.4 -> 0.00 mm
- net Net-(D4-Pad2): track 31.2 -> 0.00 mm
- net Net-(D10-Pad2): track 31.2 -> 0.00 mm
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Other:
- outline, holes or cut-outs redrawn
