File: touchL/MTCH6102_breakout.kicad_pcb (KiCad board)
At the start: 2 copper layers, 87 x 87 mm, 130 parts, among them J3 Conn_01x01, J4 Conn_01x01, J5 Conn_01x01, P1 Diamond_Edge, P10 Diamond, P11 Diamond, P12 Diamond, P13 Diamond, P14 Diamond, P15 Diamond, P16 Diamond, P17 Diamond, P18 Diamond, P19 Diamond, P2 Diamond_Edge, P20 Diamond, P21 Diamond, P22 Diamond, P23 Diamond, P24 Diamond, P25 Diamond, P26 Diamond, P27 Diamond, P28 Diamond, P29 Diamond, P3 Diamond_Edge, P30 Diamond, P31 Diamond, P32 Diamond, P33 Diamond, P34 Diamond, P35 Diamond, P36 Diamond, P37 Diamond, P38 Diamond, P39 Diamond, P4 Diamond_Edge, P40 Diamond, P41 Diamond, P42 Diamond, P43 Diamond, P44 Diamond, P45 Diamond, P46 Diamond, P47 Diamond, P48 Diamond, P49 Diamond, P5 Diamond_Edge, P50 Diamond, P51 Diamond, P52 Diamond, P53 Diamond, P54 Diamond, P6 Diamond_Edge, P7 Diamond, P8 Diamond, P9 Diamond, U2 MTCH6102_SSOP

Commit message: add pcba files
Parts:
- removed the J3 at (188.6, 167.0)
- removed the J3 at (142.9, 167.0)
- removed the J4 at (155.0, 98.4)
- removed the J4 at (154.9, 149.2)
- removed the P1 at (159.1, 103.9)
- removed the P1 at (159.1, 144.0)
- removed the P2 at (164.1, 103.9)
- removed the P2 at (164.1, 144.0)
- removed the P3 at (169.1, 103.9)
- removed the P3 at (169.1, 144.0)
- removed the P4 at (174.1, 103.9)
- removed the P4 at (174.1, 144.0)
- removed the P5 at (179.1, 144.0)
- removed the P5 at (179.1, 103.9)
- removed the P6 at (184.1, 103.9)
- removed the P6 at (184.1, 144.0)
- added J3: Conn_01x01, MountingHole:MountingHole_2.2mm_M2_Pad_Via, B.Cu at (109.3, 98.4)
- added J3: Conn_01x01, MountingHole:MountingHole_2.2mm_M2_Pad_Via, B.Cu at (155.0, 98.4)
- added J4: Conn_01x01, MountingHole:MountingHole_2.2mm_M2_Pad_Via, B.Cu at (188.6, 167.0)
- added J4: Conn_01x01, MountingHole:MountingHole_2.2mm_M2_Pad_Via, B.Cu at (155.0, 149.2)
- added P1: Diamond_Edge, Keyboard:diamond_top_edge, B.Cu at (159.2, 144.0)
- added P1: Diamond_Edge, Keyboard:diamond_top_edge, B.Cu at (159.2, 103.9)
- added P2: Diamond_Edge, Keyboard:diamond_top_edge, B.Cu at (164.2, 103.9)
- added P2: Diamond_Edge, Keyboard:diamond_top_edge, B.Cu at (164.2, 144.0)
- added P3: Diamond_Edge, Keyboard:diamond_top_edge, B.Cu at (169.2, 144.0)
- added P3: Diamond_Edge, Keyboard:diamond_top_edge, B.Cu at (169.2, 103.9)
- added P4: Diamond_Edge, Keyboard:diamond_top_edge, B.Cu at (174.2, 144.0)
- added P4: Diamond_Edge, Keyboard:diamond_top_edge, B.Cu at (174.2, 103.9)
- added P5: Diamond_Edge, Keyboard:diamond_top_edge, B.Cu at (179.2, 103.9)
- added P5: Diamond_Edge, Keyboard:diamond_top_edge, B.Cu at (179.2, 144.0)
- added P6: Diamond_Edge, Keyboard:diamond_top_edge, B.Cu at (184.2, 144.0)
- added P6: Diamond_Edge, Keyboard:diamond_top_edge, B.Cu at (184.2, 103.9)
- moved J4 76.4 mm to (142.9, 167.0)
Routing:
- net /SDA: track 222.9 -> 20.7 mm
- net /SCL: track 59.8 -> 161.6 mm
- net VCC: track 119.3 -> 68.7 mm
- net GND: track 374.1 -> 407.9 mm, vias 58 -> 60
- net /Y8: track 102.9 -> 101.3 mm
- net /Y1: track 169.7 -> 168.2 mm
- net /Y7: track 112.8 -> 111.3 mm
- net /Y3: track 152.5 -> 151.0 mm
- net /Y2: track 160.0 -> 158.5 mm
- net /Y0: track 180.0 -> 178.5 mm
- net /Y6: track 122.8 -> 121.3 mm
- net /Y4: track 142.7 -> 141.3 mm
- net /X1: track 101.4 -> 100.2 mm
- net /X5: track 130.5 -> 129.3 mm
Other:
- outline, holes or cut-outs redrawn
