File: touchR/MTCH6102_breakout_panel.kicad_pcb (KiCad board)
At the start: 2 copper layers, 87 x 85.7 mm, 130 parts, among them J3 Conn_01x01, J4 Conn_01x01, J5 Conn_01x01, P1 Diamond_Edge, P10 Diamond, P11 Diamond, P12 Diamond, P13 Diamond, P14 Diamond, P15 Diamond, P16 Diamond, P17 Diamond, P18 Diamond, P19 Diamond, P2 Diamond_Edge, P20 Diamond, P21 Diamond, P22 Diamond, P23 Diamond, P24 Diamond, P25 Diamond, P26 Diamond, P27 Diamond, P28 Diamond, P29 Diamond, P3 Diamond_Edge, P30 Diamond, P31 Diamond, P32 Diamond, P33 Diamond, P34 Diamond, P35 Diamond, P36 Diamond, P37 Diamond, P38 Diamond, P39 Diamond, P4 Diamond_Edge, P40 Diamond, P41 Diamond, P42 Diamond, P43 Diamond, P44 Diamond, P45 Diamond, P46 Diamond, P47 Diamond, P48 Diamond, P49 Diamond, P5 Diamond_Edge, P50 Diamond, P51 Diamond, P52 Diamond, P53 Diamond, P54 Diamond, P6 Diamond_Edge, P7 Diamond, P8 Diamond, P9 Diamond, U2 MTCH6102_SSOP

Commit message: add pcba files
Parts:
- removed the J3 at (109.3, 167.2)
- removed the J3 at (155.0, 167.2)
- removed the J4 at (188.6, 98.7)
- removed the J4 at (188.7, 149.5)
- removed the P1 at (159.4, 144.2)
- removed the P1 at (159.4, 104.1)
- removed the P2 at (164.4, 104.1)
- removed the P2 at (164.4, 144.2)
- removed the P3 at (169.4, 104.1)
- removed the P3 at (169.4, 144.2)
- removed the P4 at (174.4, 144.2)
- removed the P4 at (174.4, 104.1)
- removed the P5 at (179.4, 144.2)
- removed the P5 at (179.4, 104.1)
- removed the P6 at (184.4, 144.2)
- removed the P6 at (184.4, 104.1)
- added J3: Conn_01x01, MountingHole:MountingHole_2.2mm_M2_Pad_Via, F.Cu at (142.9, 98.7)
- added J3: Conn_01x01, MountingHole:MountingHole_2.2mm_M2_Pad_Via, F.Cu at (188.6, 98.7)
- added J4: Conn_01x01, MountingHole:MountingHole_2.2mm_M2_Pad_Via, F.Cu at (188.7, 149.5)
- added J4: Conn_01x01, MountingHole:MountingHole_2.2mm_M2_Pad_Via, F.Cu at (155.0, 167.2)
- added P1: Diamond_Edge, Keyboard:diamond_top_edge, B.Cu at (159.4, 104.1)
- added P1: Diamond_Edge, Keyboard:diamond_top_edge, B.Cu at (159.4, 144.2)
- added P2: Diamond_Edge, Keyboard:diamond_top_edge, B.Cu at (164.4, 144.2)
- added P2: Diamond_Edge, Keyboard:diamond_top_edge, B.Cu at (164.4, 104.1)
- added P3: Diamond_Edge, Keyboard:diamond_top_edge, B.Cu at (169.4, 144.2)
- added P3: Diamond_Edge, Keyboard:diamond_top_edge, B.Cu at (169.4, 104.1)
- added P4: Diamond_Edge, Keyboard:diamond_top_edge, B.Cu at (174.4, 104.1)
- added P4: Diamond_Edge, Keyboard:diamond_top_edge, B.Cu at (174.4, 144.2)
- added P5: Diamond_Edge, Keyboard:diamond_top_edge, B.Cu at (179.4, 104.1)
- added P5: Diamond_Edge, Keyboard:diamond_top_edge, B.Cu at (179.4, 144.2)
- added P6: Diamond_Edge, Keyboard:diamond_top_edge, B.Cu at (184.4, 104.1)
- added P6: Diamond_Edge, Keyboard:diamond_top_edge, B.Cu at (184.4, 144.2)
- moved J4 76.4 mm to (109.3, 167.2)
Routing:
- net /SDA: track 218.3 -> 14.3 mm
- net /SCL: track 24.8 -> 150.9 mm
- net VCC: track 130.5 -> 77.5 mm
- net /X0: track 138.2 -> 137.1 mm
